File: schematic/v5/TZATZIKI_v5.sch (EAGLE design)
At the start: 21 parts, among them J1 2X20-CHIP-HEADERS2X20CHIP_OFF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, U2 DS2431P

Commit message: connected audio gnd
Parts:
- added GND, P0, P1, P3, P4: SE11, solpad:SE11
Connections:
- new net N$23: J1.XIO-P1, P1.MP
- new net N$24: J1.XIO-P3, P3.MP
- new net N$25: J1.XIO-P0, P0.MP
- new net N$26: J1.XIO-P2, P4.MP
- net GND: now also GND.MP, J1.HPCOM
Changed lines of the file:
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@@
 <part name="C6" library="rcl" deviceset="C-EU" device="C0805" value="1uF"/>
 <part name="U$2" library="JKW_CHIP" deviceset="LOGO_10X10_SILK" device=""/>
+<part name="P1" library="solpad" deviceset="SE11" device=""/>
+<part name="P3" library="solpad" deviceset="SE11" device=""/>
+<part name="P0" library="solpad" deviceset="SE11" device=""/>
+<part name="P4" library="solpad" deviceset="SE11" device=""/>
+<part name="GND" library="solpad" deviceset="SE11" device=""/>
+<part name="GND10" library="supply1" deviceset="GND" device=""/>
 </parts>
 <sheets>
@@
 <instance part="C6" gate="G$1" x="132.08" y="-40.64"/>
 <instance part="U$2" gate="G$1" x="27.94" y="-35.56"/>
+<instance part="P1" gate="1" x="111.76" y="50.8"/>
+<instance part="P3" gate="1" x="116.84" y="50.8"/>
+<instance part="P0" gate="1" x="63.5" y="53.34"/>
+<instance part="P4" gate="1" x="58.42" y="53.34"/>
+<instance part="GND" gate="1" x="144.78" y="27.94"/>
+<instance part="GND10" gate="1" x="129.54" y="71.12"/>
 </instances>
 <busses>
@@
 <wire x1="167.64" y1="22.86" x2="165.1" y2="22.86" width="0.1524" layer="91"/>
 <wire x1="165.1" y1="22.86" x2="162.56" y2="22.86" width="0.1524" layer="91"/>
-<wire x1="162.56" y1="22.86" x2="137.16" y2="22.86" width="0.1524" layer="91"/>
+<wire x1="162.56" y1="22.86" x2="144.78" y2="22.86" width="0.1524" layer="91"/>
+<wire x1="144.78" y1="22.86" x2="137.16" y2="22.86" width="0.1524" layer="91"/>
 <wire x1="185.42" y1="40.64" x2="152.4" y2="40.64" width="0.1524" layer="91"/>
 <wire x1="152.4" y1="40.64" x2="137.16" y2="40.64" width="0.1524" layer="91"/>
@@
 <junction x="198.12" y="22.86"/>
 <junction x="200.66" y="22.86"/>
+<pinref part="GND" gate="1" pin="MP"/>
+<wire x1="144.78" y1="25.4" x2="144.78" y2="22.86" width="0.1524" layer="91"/>
+<junction x="144.78" y="22.86"/>
 </segment>
 <segment>
@@
 <wire x1="132.08" y1="-50.8" x2="157.48" y2="-50.8" width="0.1524" layer="91"/>
 <junction x="157.48" y="-50.8"/>
+</segment>
+<segment>
+<pinref part="J1" gate="G$1" pin="HPCOM"/>
+<wire x1="109.22" y1="58.42" x2="124.46" y2="58.42" width="0.1524" layer="91"/>
+<wire x1="124.46" y1="58.42" x2="124.46" y2="76.2" width="0.1524" layer="91"/>
+<pinref part="GND10" gate="1" pin="GND"/>
+<wire x1="124.46" y1="76.2" x2="129.54" y2="76.2" width="0.1524" layer="91"/>
+<wire x1="129.54" y1="76.2" x2="129.54" y2="73.66" width="0.1524" layer="91"/>
 </segment>
 </net>
@@
 </segment>
 </net>
+<net name="N$23" class="0">
+<segment>
+<pinref part="J1" gate="G$1" pin="XIO-P1"/>
+<wire x1="109.22" y1="48.26" x2="111.76" y2="48.26" width="0.1524" layer="91"/>
+<pinref part="P1" gate="1" pin="MP"/>
+</segment>
+</net>
+<net name="N$24" class="0">
+<segment>
+<pinref part="J1" gate="G$1" pin="XIO-P3"/>
+<wire x1="109.22" y1="45.72" x2="116.84" y2="45.72" width="0.1524" layer="91"/>
+<pinref part="P3" gate="1" pin="MP"/>
+<wire x1="116.84" y1="45.72" x2="116.84" y2="48.26" width="0.1524" layer="91"/>
+</segment>
+</net>
+<net name="N$25" class="0">
+<segment>
+<pinref part="J1" gate="G$1" pin="XIO-P0"/>
+<wire x1="76.2" y1="48.26" x2="63.5" y2="48.26" width="0.1524" layer="91"/>
+<pinref part="P0" gate="1" pin="MP"/>
+<wire x1="63.5" y1="48.26" x2="63.5" y2="50.8" width="0.1524" layer="91"/>
+</segment>
+</net>
+<net name="N$26" class="0">
+<segment>
+<pinref part="J1" gate="G$1" pin="XIO-P2"/>
+<wire x1="76.2" y1="45.72" x2="58.42" y2="45.72" width="0.1524" layer="91"/>
+<pinref part="P4" gate="1" pin="MP"/>
+<wire x1="58.42" y1="45.72" x2="58.42" y2="50.8" width="0.1524" layer="91"/>
+</segment>
+</net>

Commit message: added shutdown pin control
Connections:
- new net N$27: J1.XIO-P4, PAM1.SHND
- net N$7: no longer PAM1.SHND
Changed lines of the file:
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@@
 <instance part="GND4" gate="1" x="50.8" y="2.54"/>
 <instance part="GND5" gate="1" x="10.16" y="2.54"/>
-<instance part="U$1" gate="G$1" x="27.94" y="-27.94"/>
+<instance part="U$1" gate="G$1" x="-48.26" y="-27.94"/>
 <instance part="POWER_USB" gate="G$1" x="-20.32" y="76.2" rot="MR0"/>
 <instance part="GND18" gate="1" x="-12.7" y="71.12" rot="MR0"/>
@@
 <instance part="R2" gate="G$1" x="218.44" y="20.32" rot="MR90"/>
 <instance part="C6" gate="G$1" x="132.08" y="-40.64"/>
-<instance part="U$2" gate="G$1" x="27.94" y="-35.56"/>
+<instance part="U$2" gate="G$1" x="-48.26" y="-35.56"/>
 <instance part="P1" gate="1" x="111.76" y="50.8"/>
 <instance part="P3" gate="1" x="116.84" y="50.8"/>
@@
 <pinref part="PAM1" gate="G$1" pin="PVDD1"/>
 <wire x1="213.36" y1="-48.26" x2="213.36" y2="-30.48" width="0.1524" layer="91"/>
-<wire x1="213.36" y1="-30.48" x2="213.36" y2="-27.94" width="0.1524" layer="91"/>
-<wire x1="213.36" y1="-27.94" x2="213.36" y2="-25.4" width="0.1524" layer="91"/>
+<wire x1="213.36" y1="-30.48" x2="213.36" y2="-25.4" width="0.1524" layer="91"/>
 <wire x1="213.36" y1="-25.4" x2="200.66" y2="-25.4" width="0.1524" layer="91"/>
 <wire x1="167.64" y1="-25.4" x2="166.37" y2="-25.4" width="0.1524" layer="91"/>
@@
 <pinref part="PAM1" gate="G$1" pin="PVDD"/>
 <junction x="166.37" y="-25.4"/>
-<pinref part="PAM1" gate="G$1" pin="SHND"/>
-<wire x1="200.66" y1="-27.94" x2="213.36" y2="-27.94" width="0.1524" layer="91"/>
-<junction x="213.36" y="-27.94"/>
 <pinref part="C2" gate="G$1" pin="2"/>
 <wire x1="142.24" y1="-30.48" x2="149.86" y2="-30.48" width="0.1524" layer="91"/>
@@
 </segment>
 </net>
+<net name="N$27" class="0">
+<segment>
+<pinref part="J1" gate="G$1" pin="XIO-P4"/>
+<wire x1="76.2" y1="43.18" x2="60.96" y2="43.18" width="0.1524" layer="91"/>
+<wire x1="60.96" y1="43.18" x2="60.96" y2="-7.62" width="0.1524" layer="91"/>
+<wire x1="60.96" y1="-7.62" x2="127" y2="-7.62" width="0.1524" layer="91"/>
+<wire x1="127" y1="-7.62" x2="127" y2="-2.54" width="0.1524" layer="91"/>
+<wire x1="127" y1="-2.54" x2="203.2" y2="-2.54" width="0.1524" layer="91"/>
+<wire x1="203.2" y1="-2.54" x2="203.2" y2="-27.94" width="0.1524" layer="91"/>
+<pinref part="PAM1" gate="G$1" pin="SHND"/>
+<wire x1="203.2" y1="-27.94" x2="200.66" y2="-27.94" width="0.1524" layer="91"/>
+</segment>
+</net>

Commit message: added bat con and pwrbutton
Parts:
- added PWR-BTN, VBAT: (no value), pinhead:PINHD-1X2
Connections:
- new net N$28: J1.VBAT-EXT, VBAT.2
- new net N$29: J1.PWRON, PWR-BTN.2
- net GND: now also PWR-BTN.1, VBAT.1
Changed lines of the file:
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@@
 <part name="GND" library="solpad" deviceset="SE11" device=""/>
 <part name="GND10" library="supply1" deviceset="GND" device=""/>
+<part name="PWR-BTN" library="pinhead" deviceset="PINHD-1X2" device=""/>
+<part name="VBAT" library="pinhead" deviceset="PINHD-1X2" device=""/>
+<part name="GND11" library="supply1" deviceset="GND" device=""/>
 </parts>
 <sheets>
@@
 <instance part="GND" gate="1" x="144.78" y="27.94"/>
 <instance part="GND10" gate="1" x="129.54" y="71.12"/>
+<instance part="PWR-BTN" gate="G$1" x="17.78" y="101.6" rot="R180"/>
+<instance part="VBAT" gate="G$1" x="17.78" y="91.44" rot="R180"/>
+<instance part="GND11" gate="1" x="30.48" y="83.82" rot="MR0"/>
 </instances>
 <busses>
@@
 <wire x1="129.54" y1="76.2" x2="129.54" y2="73.66" width="0.1524" layer="91"/>
 </segment>
+<segment>
+<pinref part="PWR-BTN" gate="G$1" pin="1"/>
+<pinref part="GND11" gate="1" pin="GND"/>
+<wire x1="20.32" y1="99.06" x2="30.48" y2="99.06" width="0.1524" layer="91"/>
+<wire x1="30.48" y1="99.06" x2="30.48" y2="88.9" width="0.1524" layer="91"/>
+<pinref part="VBAT" gate="G$1" pin="1"/>
+<wire x1="30.48" y1="88.9" x2="30.48" y2="86.36" width="0.1524" layer="91"/>
+<wire x1="20.32" y1="88.9" x2="30.48" y2="88.9" width="0.1524" layer="91"/>
+<junction x="30.48" y="88.9"/>
+</segment>
 </net>
 <net name="N$2" class="0">
@@
 </segment>
 </net>
+<net name="N$28" class="0">
+<segment>
+<pinref part="J1" gate="G$1" pin="VBAT-EXT"/>
+<wire x1="45.72" y1="55.88" x2="48.26" y2="55.88" width="0.1524" layer="91"/>
+<pinref part="VBAT" gate="G$1" pin="2"/>
+<wire x1="48.26" y1="55.88" x2="48.26" y2="91.44" width="0.1524" layer="91"/>
+<wire x1="48.26" y1="91.44" x2="20.32" y2="91.44" width="0.1524" layer="91"/>
+</segment>
+</net>
+<net name="N$29" class="0">
+<segment>
+<pinref part="J1" gate="G$1" pin="PWRON"/>
+<wire x1="45.72" y1="53.34" x2="55.88" y2="53.34" width="0.1524" layer="91"/>
+<pinref part="PWR-BTN" gate="G$1" pin="2"/>
+<wire x1="55.88" y1="53.34" x2="55.88" y2="101.6" width="0.1524" layer="91"/>
+<wire x1="55.88" y1="101.6" x2="20.32" y2="101.6" width="0.1524" layer="91"/>
+</segment>
+</net>
