File: schematic/v8/TZATZIKI_v8.sch (EAGLE design)
At the start: 33 parts, among them J1 2X20-CHIP, P0 SE11, P1 SE11, P3 SE11, P4 SE11, U2 DS2431P

Commit message: added stereo poti pads
Parts:
- removed A_I, A_O: SE11, solpad:SE11
- removed SJ1: (no value), jumper:SJ
- added L_I, L_O, R_I, R_O: SE11, solpad:SE11
- added SJ3: (no value), jumper:SJ
Connections:
- removed net N$17: A_I.MP, J1.HPR, SJ1.2
- new net N$31: C4.2, R_I.MP, SJ2.2
- new net N$32: C5.2, L_I.MP, SJ3.2
- net N$15: now also L_O.MP, SJ3.1; no longer C5.2, SJ2.1
- net N$18: now also R_O.MP, SJ2.1; no longer C4.2, SJ2.2
- net N$30: now also J1.HPR; no longer A_O.MP, SJ1.1
Other:
- note removed: "Removed R1 or C5 and connect SJ2 if you want to go MONO"
- moved on the sheet: SJ2
Changed lines of the file:
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@@
 <part name="J1" library="JKW_CHIP" deviceset="2X20-CHIP" device=""/>
 <part name="R2" library="rcl" deviceset="R-EU_" device="R0805" value="10k"/>
-<part name="A_I" library="solpad" deviceset="SE11" device=""/>
-<part name="A_O" library="solpad" deviceset="SE11" device=""/>
 <part name="A_G" library="solpad" deviceset="SE11" device=""/>
 <part name="SJ2" library="jumper" deviceset="SJ" device=""/>
-<part name="SJ1" library="jumper" deviceset="SJ" device=""/>
+<part name="SJ3" library="jumper" deviceset="SJ" device=""/>
+<part name="L_I" library="solpad" deviceset="SE11" device=""/>
+<part name="L_O" library="solpad" deviceset="SE11" device=""/>
+<part name="R_I" library="solpad" deviceset="SE11" device=""/>
+<part name="R_O" library="solpad" deviceset="SE11" device=""/>
 </parts>
 <sheets>
 <sheet>
 <plain>
-<text x="248.92" y="7.62" size="1.778" layer="91">Removed R1 or C5 and
- connect SJ2 if you
-want to go MONO</text>
 </plain>
 <instances>
@@
 <instance part="J1" gate="G$1" x="60.96" y="40.64"/>
 <instance part="R2" gate="G$1" x="218.44" y="20.32" rot="MR90"/>
-<instance part="A_I" gate="1" x="215.9" y="38.1" rot="R90"/>
-<instance part="A_O" gate="1" x="215.9" y="27.94" rot="R90"/>
 <instance part="A_G" gate="1" x="152.4" y="27.94"/>
-<instance part="SJ2" gate="1" x="251.46" y="0"/>
-<instance part="SJ1" gate="1" x="218.44" y="33.02" rot="R90"/>
+<instance part="SJ2" gate="1" x="231.14" y="-10.16" rot="R90"/>
+<instance part="SJ3" gate="1" x="233.68" y="-10.16" rot="R90"/>
+<instance part="L_I" gate="1" x="256.54" y="5.08"/>
+<instance part="L_O" gate="1" x="261.62" y="5.08"/>
+<instance part="R_I" gate="1" x="243.84" y="5.08"/>
+<instance part="R_O" gate="1" x="248.92" y="5.08"/>
 </instances>
 <busses>
@@
 <pinref part="PAM1" gate="G$1" pin="INL"/>
 <junction x="166.37" y="-33.02"/>
-<wire x1="233.68" y1="-45.72" x2="233.68" y2="0" width="0.1524" layer="91"/>
-<wire x1="233.68" y1="0" x2="233.68" y2="2.54" width="0.1524" layer="91"/>
-<wire x1="233.68" y1="2.54" x2="228.6" y2="2.54" width="0.1524" layer="91"/>
-<pinref part="C5" gate="G$1" pin="2"/>
-<wire x1="228.6" y1="2.54" x2="228.6" y2="5.08" width="0.1524" layer="91"/>
-<pinref part="SJ2" gate="1" pin="1"/>
-<wire x1="233.68" y1="0" x2="246.38" y2="0" width="0.1524" layer="91"/>
-<junction x="233.68" y="0"/>
-</segment>
-</net>
-<net name="N$17" class="0">
-<segment>
-<wire x1="109.22" y1="55.88" x2="132.08" y2="55.88" width="0.1524" layer="91"/>
-<wire x1="132.08" y1="55.88" x2="132.08" y2="60.96" width="0.1524" layer="91"/>
-<wire x1="132.08" y1="60.96" x2="218.44" y2="60.96" width="0.1524" layer="91"/>
-<pinref part="J1" gate="G$1" pin="HPR"/>
-<pinref part="A_I" gate="1" pin="MP"/>
-<wire x1="218.44" y1="38.1" x2="218.44" y2="60.96" width="0.1524" layer="91"/>
-<junction x="218.44" y="38.1"/>
-<pinref part="SJ1" gate="1" pin="2"/>
+<wire x1="233.68" y1="-45.72" x2="233.68" y2="-17.78" width="0.1524" layer="91"/>
+<pinref part="SJ3" gate="1" pin="1"/>
+<wire x1="233.68" y1="-17.78" x2="233.68" y2="-15.24" width="0.1524" layer="91"/>
+<wire x1="233.68" y1="-17.78" x2="261.62" y2="-17.78" width="0.1524" layer="91"/>
+<pinref part="L_O" gate="1" pin="MP"/>
+<wire x1="261.62" y1="-17.78" x2="261.62" y2="2.54" width="0.1524" layer="91"/>
+<junction x="233.68" y="-17.78"/>
 </segment>
 </net>
@@
 <pinref part="PAM1" gate="G$1" pin="INR"/>
 <wire x1="231.14" y1="-33.02" x2="200.66" y2="-33.02" width="0.1524" layer="91"/>
-<pinref part="C4" gate="G$1" pin="2"/>
-<wire x1="218.44" y1="5.08" x2="218.44" y2="-2.54" width="0.1524" layer="91"/>
-<wire x1="218.44" y1="-2.54" x2="231.14" y2="-2.54" width="0.1524" layer="91"/>
-<wire x1="231.14" y1="-2.54" x2="231.14" y2="-33.02" width="0.1524" layer="91"/>
-<wire x1="231.14" y1="-2.54" x2="259.08" y2="-2.54" width="0.1524" layer="91"/>
-<wire x1="259.08" y1="-2.54" x2="259.08" y2="0" width="0.1524" layer="91"/>
-<pinref part="SJ2" gate="1" pin="2"/>
-<wire x1="259.08" y1="0" x2="256.54" y2="0" width="0.1524" layer="91"/>
-<junction x="231.14" y="-2.54"/>
+<pinref part="SJ2" gate="1" pin="1"/>
+<wire x1="231.14" y1="-15.24" x2="231.14" y2="-33.02" width="0.1524" layer="91"/>
+<wire x1="231.14" y1="-15.24" x2="248.92" y2="-15.24" width="0.1524" layer="91"/>
+<pinref part="R_O" gate="1" pin="MP"/>
+<wire x1="248.92" y1="-15.24" x2="248.92" y2="2.54" width="0.1524" layer="91"/>
+<junction x="231.14" y="-15.24"/>
 </segment>
 </net>
@@
 </segment>
 </net>
+<net name="N$31" class="0">
+<segment>
+<pinref part="SJ2" gate="1" pin="2"/>
+<wire x1="231.14" y1="-2.54" x2="231.14" y2="-5.08" width="0.1524" layer="91"/>
+<pinref part="C4" gate="G$1" pin="2"/>
+<wire x1="218.44" y1="5.08" x2="218.44" y2="-2.54" width="0.1524" layer="91"/>
+<wire x1="218.44" y1="-2.54" x2="231.14" y2="-2.54" width="0.1524" layer="91"/>
+<wire x1="231.14" y1="-2.54" x2="243.84" y2="-2.54" width="0.1524" layer="91"/>
+<pinref part="R_I" gate="1" pin="MP"/>
+<wire x1="243.84" y1="-2.54" x2="243.84" y2="2.54" width="0.1524" layer="91"/>
+<junction x="231.14" y="-2.54"/>
+</segment>
+</net>
+<net name="N$32" class="0">
+<segment>
+<pinref part="C5" gate="G$1" pin="2"/>
+<wire x1="228.6" y1="2.54" x2="228.6" y2="5.08" width="0.1524" layer="91"/>
+<wire x1="233.68" y1="2.54" x2="228.6" y2="2.54" width="0.1524" layer="91"/>
+<wire x1="233.68" y1="-5.08" x2="233.68" y2="0" width="0.1524" layer="91"/>
+<pinref part="SJ3" gate="1" pin="2"/>
+<wire x1="233.68" y1="0" x2="233.68" y2="2.54" width="0.1524" layer="91"/>
+<wire x1="233.68" y1="0" x2="256.54" y2="0" width="0.1524" layer="91"/>
+<pinref part="L_I" gate="1" pin="MP"/>
+<wire x1="256.54" y1="0" x2="256.54" y2="2.54" width="0.1524" layer="91"/>
+<junction x="233.68" y="0"/>
+</segment>
+</net>
 <net name="N$30" class="0">
 <segment>
-<pinref part="A_O" gate="1" pin="MP"/>
-<junction x="218.44" y="27.94"/>
-<pinref part="SJ1" gate="1" pin="1"/>
+<wire x1="109.22" y1="55.88" x2="132.08" y2="55.88" width="0.1524" layer="91"/>
+<wire x1="132.08" y1="55.88" x2="132.08" y2="60.96" width="0.1524" layer="91"/>
+<wire x1="132.08" y1="60.96" x2="218.44" y2="60.96" width="0.1524" layer="91"/>
+<pinref part="J1" gate="G$1" pin="HPR"/>
+<wire x1="218.44" y1="25.4" x2="218.44" y2="60.96" width="0.1524" layer="91"/>
 <pinref part="R2" gate="G$1" pin="2"/>
-<wire x1="218.44" y1="25.4" x2="218.44" y2="27.94" width="0.1524" layer="91"/>
 </segment>
 </net>
@@
 </schematic>
 </drawing>
-<compatibility>
-<note version="6.3" minversion="6.2.2" severity="warning">
-Since Version 6.2.2 text objects can contain more than one line,
-which will not be processed correctly with this version.
-</note>
-</compatibility>
 </eagle>

Commit message: added stereo pot, holes 0.9 todo
Parts:
- added A_G1: SE11, solpad:SE11
Connections:
- net GND: now also A_G1.MP
Other:
- moved on the sheet: A_G
Changed lines of the file:
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@@
 <part name="R_I" library="solpad" deviceset="SE11" device=""/>
 <part name="R_O" library="solpad" deviceset="SE11" device=""/>
+<part name="A_G1" library="solpad" deviceset="SE11" device=""/>
 </parts>
 <sheets>
@@
 <instance part="J1" gate="G$1" x="60.96" y="40.64"/>
 <instance part="R2" gate="G$1" x="218.44" y="20.32" rot="MR90"/>
-<instance part="A_G" gate="1" x="152.4" y="27.94"/>
+<instance part="A_G" gate="1" x="281.94" y="5.08"/>
 <instance part="SJ2" gate="1" x="231.14" y="-10.16" rot="R90"/>
 <instance part="SJ3" gate="1" x="233.68" y="-10.16" rot="R90"/>
@@
 <instance part="R_I" gate="1" x="243.84" y="5.08"/>
 <instance part="R_O" gate="1" x="248.92" y="5.08"/>
+<instance part="A_G1" gate="1" x="271.78" y="5.08"/>
 </instances>
 <busses>
@@
 <wire x1="167.64" y1="22.86" x2="165.1" y2="22.86" width="0.1524" layer="91"/>
 <wire x1="165.1" y1="22.86" x2="162.56" y2="22.86" width="0.1524" layer="91"/>
-<wire x1="162.56" y1="22.86" x2="152.4" y2="22.86" width="0.1524" layer="91"/>
-<wire x1="152.4" y1="22.86" x2="144.78" y2="22.86" width="0.1524" layer="91"/>
+<wire x1="162.56" y1="22.86" x2="144.78" y2="22.86" width="0.1524" layer="91"/>
 <wire x1="144.78" y1="22.86" x2="137.16" y2="22.86" width="0.1524" layer="91"/>
 <wire x1="180.34" y1="40.64" x2="152.4" y2="40.64" width="0.1524" layer="91"/>
@@
 <wire x1="144.78" y1="25.4" x2="144.78" y2="22.86" width="0.1524" layer="91"/>
 <junction x="144.78" y="22.86"/>
-<pinref part="A_G" gate="1" pin="MP"/>
-<wire x1="152.4" y1="25.4" x2="152.4" y2="22.86" width="0.1524" layer="91"/>
-<junction x="152.4" y="22.86"/>
 </segment>
 <segment>
@@
 <wire x1="223.52" y1="-22.86" x2="223.52" y2="-20.32" width="0.1524" layer="91"/>
 <junction x="223.52" y="-20.32"/>
+<pinref part="A_G1" gate="1" pin="MP"/>
+<wire x1="248.92" y1="-20.32" x2="271.78" y2="-20.32" width="0.1524" layer="91"/>
+<wire x1="271.78" y1="-20.32" x2="271.78" y2="2.54" width="0.1524" layer="91"/>
+<wire x1="271.78" y1="-20.32" x2="281.94" y2="-20.32" width="0.1524" layer="91"/>
+<wire x1="281.94" y1="-20.32" x2="281.94" y2="2.54" width="0.1524" layer="91"/>
+<junction x="271.78" y="-20.32"/>
+<pinref part="A_G" gate="1" pin="MP"/>
 </segment>
 <segment>
